Commit message: save

File: models/leaders/papras_7dof_leaders_table.urdf (robot description, URDF)
Before this commit: robot papras_leaders, 11 links, 10 joints
Links:
- added link robot2/base_link, mass 0.218376911489293; collision mesh filename=assets/leaders/base_link.stl; visual mesh filename=assets/leaders/base_link.stl
- added link robot2/end_effector_link, mass 0.001; visual box size=0.01 0.01 0.01
- added link robot2/handle, mass 0.0792318961261061; collision mesh filename=assets/leaders/handle.stl; visual mesh filename=assets/leaders/handle.stl
- added link robot2/link1, mass 0.0184621083060345; collision mesh filename=assets/leaders/papras_7dof/link1.stl; visual mesh filename=assets/leaders/papras_7dof/link1.stl
- added link robot2/link2, mass 0.0814342847713924; collision mesh filename=assets/leaders/papras_7dof/link2.stl; visual mesh filename=assets/leaders/papras_7dof/link2.stl
- added link robot2/link3, mass 0.0654267493288997; collision mesh filename=assets/leaders/papras_7dof/link3.stl; visual mesh filename=assets/leaders/papras_7dof/link3.stl
- added link robot2/link4, mass 0.0269077999710614; collision mesh filename=assets/leaders/papras_7dof/link4.stl; visual mesh filename=assets/leaders/papras_7dof/link4.stl
- added link robot2/link5, mass 0.0354352330271564; collision mesh filename=assets/leaders/papras_7dof/link5.stl; visual mesh filename=assets/leaders/papras_7dof/link5.stl
- added link robot2/link6, mass 0.0465686690697251; collision mesh filename=assets/leaders/papras_7dof/link6.stl; visual mesh filename=assets/leaders/papras_7dof/link6.stl
- added link robot2/trigger, mass 0.0113373798119285; collision mesh filename=assets/leaders/trigger.stl; visual mesh filename=assets/leaders/trigger.stl
Joints:
- added joint robot2/end_effector_joint: type fixed, parent robot2/handle, child robot2/end_effector_link, origin xyz=0.0 0.0 0.0 rpy=0 -1.57 1.57
- added joint robot2/gripper: type revolute, parent robot2/handle, child robot2/trigger, origin xyz=0.0154268 0 0.0226837 rpy=0.0 0 0.000, axis 0 -1 0, limit lower=0 upper=1.2 effort=1 velocity=3.15
- added joint robot2/joint1: type revolute, parent robot2/base_link, child robot2/link1, origin xyz=-0.000125 0.0022 0.099 rpy=1.5708 0 0, axis 0 1 0, limit lower=-3.141592653589793 upper=3.141592653589793 effort=1 velocity=3.15
- added joint robot2/joint2: type revolute, parent robot2/link1, child robot2/link2, origin xyz=0 0.029 0 rpy=3.1416 0 3.1416, axis 0 0 -1, limit lower=-3.141592653589793 upper=3.141592653589793 effort=1 velocity=3.15
- added joint robot2/joint3: type revolute, parent robot2/link2, child robot2/link3, origin xyz=-0.0001 0.10079 0 rpy=1.5708 1.5708 0, axis 0 0 -1, limit lower=-3.141592653589793 upper=3.141592653589793 effort=1 velocity=3.15
- added joint robot2/joint4: type revolute, parent robot2/link3, child robot2/link4, origin xyz=0 0.01952 -0.070988 rpy=1.5708 -1.5708 0, axis 0 -1 0, limit lower=-3.141592653589793 upper=3.141592653589793 effort=1 velocity=3.15
- added joint robot2/joint5: type revolute, parent robot2/link4, child robot2/link5, origin xyz=-0.01952 0 -0.12037 rpy=0 0 -1.5708, axis 0 0 -1, limit lower=-3.141592653589793 upper=3.141592653589793 effort=1 velocity=3.15
- added joint robot2/joint6: type revolute, parent robot2/link5, child robot2/link6, origin xyz=0 0 -0.0475000000000001 rpy=0 0 1.5708, axis 0 -1 0, limit lower=-3.141592653589793 upper=3.141592653589793 effort=1 velocity=3.15
- added joint robot2/joint7: type revolute, parent robot2/link6, child robot2/handle, origin xyz=0 1E-05 -0.076464 rpy=3.141592653589793 0.05236 1.576, axis 0.052336 0 0.99863, limit lower=-3.141592653589793 upper=3.141592653589793 effort=1 velocity=3.15
- added joint robot2/world_joint: type fixed, parent world, child robot2/base_link, origin xyz=0.2601 -0.33435 -0.05189 rpy=0 0 0, axis 0 0 0
- joint robot1/world_joint: origin xyz=0 0 0 rpy=0 0 0 -> xyz=0.2599 0.33455 -0.05189 rpy=0 0 0
