Commit message: visionpro added, need to check with hw

File: models/PAPRAS/papras_7dof/papras_7dof.urdf (robot description, URDF)
Before this commit: robot simple_robot, 18 links, 17 joints
Links:
- added link robot1/wrist_link
Joints:
- added joint robot1/wrist_joint: type fixed, parent robot1/end_link, child robot1/wrist_link, origin xyz=0.006 0.0 0.0 rpy=0 0 0

File: models/PAPRAS/papras_7dof_2arm_table/papras_7dof_2arm_table.urdf (robot description, URDF)
Before this commit: robot teleop_table, 34 links, 33 joints
Links:
- added link robot3/wrist_link
- added link robot4/wrist_link
Joints:
- added joint robot3/wrist_joint: type fixed, parent robot3/end_link, child robot3/wrist_link, origin xyz=0.006 0.0 0.0 rpy=0 0 0
- added joint robot4/wrist_joint: type fixed, parent robot4/end_link, child robot4/wrist_link, origin xyz=0.006 0.0 0.0 rpy=0 0 0

Commit message: workwork

File: models/PAPRAS/papras_7dof/papras_7dof.urdf (robot description, URDF)
Before this commit: robot simple_robot, 19 links, 18 joints
Links:
- added link robot1/hand_link
Joints:
- added joint robot1/hand_joint: type fixed, parent robot1/gripper_main_link, child robot1/hand_link, origin xyz=0.0 0.0 0.10 rpy=3.141592653589793 -1.5707963267948966 0

File: models/PAPRAS/papras_7dof_2arm_table/papras_7dof_2arm_table.urdf (robot description, URDF)
Before this commit: robot teleop_table, 36 links, 35 joints
Links:
- added link robot3/hand_link
- added link robot4/hand_link
Joints:
- added joint robot3/hand_joint: type fixed, parent robot3/gripper_main_link, child robot3/hand_link, origin xyz=0.0 0.0 0.10 rpy=3.141592653589793 -1.5707963267948966 0
- added joint robot4/hand_joint: type fixed, parent robot4/gripper_main_link, child robot4/hand_link, origin xyz=0.0 0.0 0.10 rpy=3.141592653589793 -1.5707963267948966 0
